File: ecad/60_keyboard.brd (EAGLE design)
At the start: 286.1 x 95.2 mm, 149 parts, among them J1 USB-C, SW1 TACTILE, Y2 CRYSTAL

Commit message: ecad, gebers
Parts:
- removed D64: (no value), Components:SOD-123
- removed D65: PRTR5V0U2X,215, PRTR5V0U2X_215:SOT143B
- removed F1: 500mA, 0686F0500-01:FUSC1608X60N
- removed ISP1: AVRISP-6, adafruit:AVRISP
- removed R5, R6: 5.1k, Components:R0805
- removed U$64: KEYSWITCH-PLAIN-MXHSPCB-1U, Keyboard:MXHSPCB-1U
- added SV1: (no value), con-lstb:MA06-1
- J1: value USB-C -> USB-CON; device USB4085-GF-A_REVA4:GCT_USB4085-GF-A_REVA4 -> 690-005-299-043:EDAC_690-005-299-043
- R3, R4: device Components:R0805 -> RMCF0805JT22R0:RESC2012X65N
- U$58: value KEYSWITCH-PLAIN-MXHSPCB-1U -> KEYSWITCH-PLAIN-MXHSPCB-6.25U-FLIPPED; device Keyboard:MXHSPCB-1U -> Keyboard:MXHSPCB-6.25U-FLIPPED
- U$59: value KEYSWITCH-PLAIN-MXHS-6.25U-FLIPPED -> KEYSWITCH-PLAIN-MXHSPCB-1U; device Keyboard:MXHS-6.25U-FLIPPED -> Keyboard:MXHSPCB-1U
- moved U$55 265.2 mm to (11.9, 9.53)
- moved D55 250.0 mm to (19.6, 6.53), turned to 180 degrees
- moved C2 165.7 mm to (159.2, 5.75), flipped to the bottom, turned to 180 degrees
- moved Y2 159.5 mm to (153.7, 6.50), flipped to the bottom
- moved C7 158.3 mm to (156.2, 19.8), flipped to the bottom, turned to 270 degrees
- moved C1 154.7 mm to (153.3, 11.0), flipped to the bottom, turned to 180 degrees
- moved C6 153.8 mm to (152.7, 19.8), flipped to the bottom, turned to 270 degrees
- moved C5 149.5 mm to (149.2, 19.8), flipped to the bottom, turned to 270 degrees
- moved R4 147.4 mm to (10.8, 91.2), flipped to the bottom, turned to 90 degrees
- moved C4 145.3 mm to (145.7, 19.8), flipped to the bottom, turned to 270 degrees
- moved R3 144.9 mm to (27.2, 91.2), flipped to the bottom, turned to 90 degrees
- moved C3 143.4 mm to (142.2, 19.8), flipped to the bottom, turned to 270 degrees
- moved J1 134.3 mm to (19.0, 92.0), flipped to the bottom, turned to 180 degrees
- moved D58 86.6 mm to (138.7, 6.53), turned to 180 degrees
- moved D59 84.1 mm to (207.7, 6.53), turned to 180 degrees
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Connections:
- removed net DN: D65.3, J1.A7, J1.B7, R4.2
- removed net DP: D65.2, J1.A6, J1.B6, R3.2
- removed net N$64 (its old number): D64.A, U$64.MX2
- removed net N$66: J1.A5, R6.2
- removed net VCC: D65.4, F1.1, J1.A4, J1.A9, J1.B4, J1.B9
- new net N$59: J1.2, R4.2
- net 5V: now also J1.1, SV1.6; no longer F1.2, ISP1.2
- net COL1: now also U$55.MX1, U$65.19; no longer U$56.MX1, U$65.31
- net COL10: now also U$60.MX1, U$65.27; no longer U$65.8
- net COL11: now also U$61.MX1, U$65.39; no longer U$65.36
- net COL12: now also U$62.MX1, U$65.38; no longer U$65.37
- net COL13: now also U$63.MX1, U$65.37; no longer U$65.38
- net COL14: now also U$65.36; no longer U$55.MX1, U$65.39
- net COL2: now also U$56.MX1, U$65.20; no longer U$57.MX1, U$65.27
- net COL3: now also U$57.MX1, U$65.21; no longer U$58.MX1, U$65.1
- net COL4: no longer U$59.MX1
- net COL5: no longer U$60.MX1
- net COL6: now also U$58.MX1; no longer U$61.MX1
- net COL7: now also U$65.31; no longer U$62.MX1, U$65.12
- net COL8: now also U$65.25; no longer U$63.MX1, U$65.26
- net COL9: now also U$59.MX1, U$65.26; no longer U$64.MX1, U$65.32
- net GND: now also J1.5, J1.S1, J1.S2, J1.S3, J1.S4, SV1.1; no longer D65.1, ISP1.6, J1.A1, J1.A12, J1.B1, J1.B12, J1.P1, J1.P2, J1.P3, J1.P4, R5.1, R6.1
- net MISO: now also SV1.2; no longer ISP1.1
- net MOSI: now also SV1.3; no longer ISP1.4
- net N$65: now also J1.3, R3.2; no longer J1.B5, R5.2
- net RESET: now also SV1.5; no longer ISP1.5
- net ROW1: now also U$65.40; no longer U$65.20
- net ROW2: now also U$65.41; no longer U$65.21
- net ROW3: now also U$65.1; no longer U$65.19
- net ROW4: now also U$65.32; no longer D55.C, U$65.18
- net ROW5: now also D55.C, U$65.12; no longer D64.C, U$65.25
- net SCLK: now also SV1.4; no longer ISP1.3
Routing:
- net ROW1: track 0.00 -> 375.4 mm, vias 0 -> 14
- net ROW2: track 0.00 -> 337.9 mm, vias 0 -> 14
- net 5V: track 0.00 -> 332.3 mm, vias 0 -> 7
- net ROW3: track 0.00 -> 307.2 mm, vias 0 -> 13
- net ROW4: track 0.00 -> 304.5 mm, vias 0 -> 14
- net ROW5: track 0.00 -> 287.1 mm, vias 0 -> 6
- net COL1: track 0.00 -> 260.4 mm
- net COL2: track 0.00 -> 228.9 mm, vias 0 -> 2
- net D-: track 0.00 -> 221.9 mm, vias 0 -> 4
- net D+: track 0.00 -> 220.3 mm, vias 0 -> 4
- net COL3: track 0.00 -> 211.9 mm, vias 0 -> 2
- net COL13: track 0.00 -> 209.7 mm, vias 0 -> 2
- net COL14: track 0.00 -> 201.0 mm, vias 0 -> 2
- net COL12: track 0.00 -> 191.9 mm, vias 0 -> 2
- net COL11: track 0.00 -> 167.7 mm, vias 0 -> 2
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- added copper zone on layer 1, net GND
- added copper zone on layer 16, net GND
Other:
- board size 286.1 x 95.2 mm -> 285.8 x 97.2 mm
- board text added: "5V"
- board text added: "ATMEGA32U4"
- board text added: "C1"
- board text added: "C2"
- board text added: "C3"
- board text added: "C4"
- board text added: "C5"
- board text added: "C6"
- board text added: "C7"
- board text added: "C8"
- board text added: "Crystal"
- board text added: "R1"
- board text added: "R2"
- board text added: "USB-CON"
- board text removed: "VCC"
