File: ecad/60_keyboard.sch (EAGLE design)
At the start: 149 parts, among them J1 USB-C, SW1 TACTILE, Y2 CRYSTAL

Commit message: ecad, gebers
Parts:
- removed D64: (no value), Components:DIODE-SOD-123
- removed D65: PRTR5V0U2X,215, PRTR5V0U2X_215:PRTR5V0U2X,215
- removed F1: 500mA, 0686F0500-01:0686F0500-01
- removed ISP1: AVRISP-6, adafruit:AVRISP-6
- removed R5, R6: 5.1k, Components:RESISTOR-0805
- removed U$64: KEYSWITCH-PLAIN-MXHSPCB-1U, Keyboard:KEYSWITCH-PLAIN-MXHSPCB-1U
- added SV1: (no value), con-lstb:MA06-1
- J1: value USB-C -> USB-CON; device USB4085-GF-A_REVA4:USB4085-GF-A_REVA4 -> 690-005-299-043:690-005-299-043
- R3, R4: device Components:RESISTOR-0805 -> RMCF0805JT22R0:RMCF0805JT22R0
- U$58: value KEYSWITCH-PLAIN-MXHSPCB-1U -> KEYSWITCH-PLAIN-MXHSPCB-6.25U-FLIPPED; device Keyboard:KEYSWITCH-PLAIN-MXHSPCB-1U -> Keyboard:KEYSWITCH-PLAIN-MXHSPCB-6.25U-FLIPPED
- U$59: value KEYSWITCH-PLAIN-MXHS-6.25U-FLIPPED -> KEYSWITCH-PLAIN-MXHSPCB-1U; device Keyboard:KEYSWITCH-PLAIN-MXHS-6.25U-FLIPPED -> Keyboard:KEYSWITCH-PLAIN-MXHSPCB-1U
Connections:
- removed net DN: D65.P$3, J1.DN1, J1.DN2, R4.2
- removed net DP: D65.P$2, J1.DP1, J1.DP2, R3.2
- removed net N$64 (its old number): D64.A, U$64.P1
- removed net N$66: J1.CC1, R6.2
- removed net VCC: D65.P$4, F1.1, J1.VBUS
- new net N$59: J1.D-, R4.2
- net 5V: now also J1.VCC, SV1.6; no longer F1.2, ISP1.VCC
- net COL1: now also U$55.P0, U$65.PD1(SDA/INT1); no longer U$56.P0, U$65.PC6(OC3A/!OC4A)
- net COL10: now also U$60.P0, U$65.PD7(T0/OC4D/ADC10); no longer U$65.PB0(SS/PCINT0)
- net COL11: now also U$61.P0, U$65.PF4(ADC4/TCK); no longer U$65.PF7(ADC7/TDI)
- net COL12: now also U$62.P0, U$65.PF5(ADC5/TMS); no longer U$65.PF6(ADC6/TDO)
- net COL13: now also U$63.P0, U$65.PF6(ADC6/TDO); no longer U$65.PF5(ADC5/TMS)
- net COL14: now also U$65.PF7(ADC7/TDI); no longer U$55.P0, U$65.PF4(ADC4/TCK)
- net COL2: now also U$56.P0, U$65.PD2(RXD1/INT2); no longer U$57.P0, U$65.PD7(T0/OC4D/ADC10)
- net COL3: now also U$57.P0, U$65.PD3(TXD1/INT3); no longer U$58.P0, U$65.PE6(INT.6/AIN0)
- net COL4: no longer U$59.P0
- net COL5: no longer U$60.P0
- net COL6: now also U$58.P0; no longer U$61.P0
- net COL7: now also U$65.PC6(OC3A/!OC4A); no longer U$62.P0, U$65.PB7(PCINT7/OC0A/OC1C/!RTS)
- net COL8: now also U$65.PD4(ICP1/ADC8); no longer U$63.P0, U$65.PD6(T1/ADC9/!OC4D)
- net COL9: now also U$59.P0, U$65.PD6(T1/ADC9/!OC4D); no longer U$64.P0, U$65.PC7(ICP3/CLK0/OC4A)
- net GND: now also J1.SHIELD, SV1.1; no longer D65.P$1, ISP1.GND, J1.SHELL, R5.1, R6.1
- net MISO: now also SV1.2; no longer ISP1.MISO
- net MOSI: now also SV1.3; no longer ISP1.MOSI
- net N$65: now also J1.D+, R3.2; no longer J1.CC2, R5.2
- net RESET: now also SV1.5; no longer ISP1.RST
- net ROW1: now also U$65.PF1(ADC1); no longer U$65.PD2(RXD1/INT2)
- net ROW2: now also U$65.PF0(ADC0); no longer U$65.PD3(TXD1/INT3)
- net ROW3: now also U$65.PE6(INT.6/AIN0); no longer U$65.PD1(SDA/INT1)
- net ROW4: now also U$65.PC7(ICP3/CLK0/OC4A); no longer D55.C, U$65.PD0(OC0B/SCL/INT0)
- net ROW5: now also D55.C, U$65.PB7(PCINT7/OC0A/OC1C/!RTS); no longer D64.C, U$65.PD4(ICP1/ADC8)
- net SCLK: now also SV1.4; no longer ISP1.SCK
Other:
- moved on the sheet: D55, D56, D57, D58, D59, D60, D61, D62, D63, U$55, U$56, U$57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
